File: 555SynthModule.kicad_pcb (KiCad board)
At the start: 2 copper layers, 64.8 x 34.3 mm, 32 parts, among them J1 Conn_01x09_Male, Q1 2N3904, Q2 2N3904, Q3 2N3904, Q4 2N3904, Q5 2N3904, U1 NE555P, U2 LM741

Commit message: Updated gerbers, minor changes
Connections:
- net /ENABLE renamed /DISABLE
Other:
- board text added: "555 Oscillator - Zach Baldwin 2020"
- board text added: "DE"
- board text removed: "EN"
