File: 555SynthModule.sch (KiCad schematic (older format))
At the start: 32 parts, among them J1 Conn_01x09_Male, Q1 2N3904, Q2 2N3904, Q3 2N3904, Q4 2N3904, Q5 2N3904, U1 NE555P, U2 LM741

Commit message: Updated gerbers, minor changes
Parts:
- C1: value C -> 0.8uF
- C2: value C -> 0.4uF
- C4: value C -> 0.2uF
- C5, C6: value C -> 0.1uF
Connections:
- net ENABLE renamed DISABLE
Changed lines of the file:
@@
 U 1 1 5FBBE865
 P 4300 4050
-F 0 "C6" H 4415 4096 50  0000 L CNN
-F 1 "C" H 4415 4005 50  0000 L CNN
+F 0 "C6" H 4350 3950 50  0000 L CNN
+F 1 "0.1uF" H 4350 3850 50  0000 L CNN
 F 2 "Capacitor_THT:C_Disc_D4.3mm_W1.9mm_P5.00mm" H 4338 3900 50  0001 C CNN
 F 3 "~" H 4300 4050 50  0001 C CNN
@@
 U 1 1 5FC18B6C
 P 2700 4050
-F 0 "C1" H 2815 4096 50  0000 L CNN
-F 1 "C" H 2815 4005 50  0000 L CNN
+F 0 "C1" H 2750 3950 50  0000 L CNN
+F 1 "0.8uF" H 2750 3850 50  0000 L CNN
 F 2 "Capacitor_THT:C_Disc_D4.3mm_W1.9mm_P5.00mm" H 2738 3900 50  0001 C CNN
 F 3 "~" H 2700 4050 50  0001 C CNN
@@
 U 1 1 5FC195CD
 P 3100 4050
-F 0 "C2" H 3215 4096 50  0000 L CNN
-F 1 "C" H 3215 4005 50  0000 L CNN
+F 0 "C2" H 3150 3950 50  0000 L CNN
+F 1 "0.4uF" H 3150 3850 50  0000 L CNN
 F 2 "Capacitor_THT:C_Disc_D4.3mm_W1.9mm_P5.00mm" H 3138 3900 50  0001 C CNN
 F 3 "~" H 3100 4050 50  0001 C CNN
@@
 U 1 1 5FC1A03F
 P 3500 4050
-F 0 "C4" H 3615 4096 50  0000 L CNN
-F 1 "C" H 3615 4005 50  0000 L CNN
+F 0 "C4" H 3550 3950 50  0000 L CNN
+F 1 "0.2uF" H 3550 3850 50  0000 L CNN
 F 2 "Capacitor_THT:C_Disc_D4.3mm_W1.9mm_P5.00mm" H 3538 3900 50  0001 C CNN
 F 3 "~" H 3500 4050 50  0001 C CNN
@@
 U 1 1 5FC1AB71
 P 3900 4050
-F 0 "C5" H 4015 4096 50  0000 L CNN
-F 1 "C" H 4015 4005 50  0000 L CNN
+F 0 "C5" H 3950 3950 50  0000 L CNN
+F 1 "0.1uF" H 3950 3850 50  0000 L CNN
 F 2 "Capacitor_THT:C_Disc_D4.3mm_W1.9mm_P5.00mm" H 3938 3900 50  0001 C CNN
 F 3 "~" H 3900 4050 50  0001 C CNN
@@
 Tuning
 Text Label 6050 4050 0    50   ~ 0
-ENABLE
+DISABLE
 Text Label 6050 4500 0    50   ~ 0
 RANGE0
