File: Arduino_MIDI_Device/ArduinoMicroDualRailBoard.kicad_pcb (KiCad board)
At the start: 2 copper layers, 135.3 x 92.7 mm, 59 parts, among them J1 Conn_01x20_Male, J10 Conn_01x02_Male, J2 Screw_Terminal_01x03, J3 Conn_01x20_Male, J4 Conn_01x20_Male, J5 Screw_Terminal_01x03, J6 Conn_01x20_Male, J7 SDS-50J, J8 SDS-50J, J9 Screw_Terminal_01x03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

Commit message: Resolved Issue #1 with MIDI connector direction
Parts:
- moved J7 17.4 mm to (107.3, 65.4), turned to 180 degrees
- moved J8 16.3 mm to (135.3, 65.4), turned to 180 degrees
- moved R7 12.7 mm to (134.0, 73.7), turned to 180 degrees
- moved C15 8.81 mm to (116.2, 73.7), turned to 270 degrees
- moved C13 5.08 mm to (122.6, 73.7), turned to 270 degrees
Routing:
- net Net-(J7-Pad4): track 35.6 -> 16.1 mm
- net Net-(C15-Pad1): track 25.4 -> 8.91 mm
- net Net-(J8-Pad4): track 19.5 -> 7.32 mm
- net Net-(C13-Pad1): track 26.2 -> 33.7 mm
- net Net-(D9-Pad2): track 38.5 -> 31.6 mm
- net Net-(J8-Pad5): track 19.5 -> 13.6 mm
- net +5V: track 185.3 -> 183.6 mm
