File: EnvelopeGenerator/EnvelopeGenerator.kicad_pcb (KiCad board)
At the start: 2 copper layers, 49.5 x 97.8 mm, 49 parts, among them J1 Conn_01x02_Male, J2 Conn_01x03_Male, J3 Conn_01x09_Male, U1 L7812, U2 L7912, U3 AS3310, U4 LM741, U5 AS3360

Commit message: Fixed C13 annotation, updated PCB
Parts:
- renumbered R6 to C13
