File: 555_Synth_Module/555SynthModule.kicad_pcb (KiCad board)
At the start: 2 copper layers, 64.8 x 34.3 mm, 32 parts, among them J1 Conn_01x09_Male, Q1 2N3904, Q2 2N3904, Q3 2N3904, Q4 2N3904, Q5 2N3904, U1 NE555P, U2 LM741

Commit message: Resolved Issue #3 Also: * Added output cap to 555 modules * EnvelopeFilter now has an output cap
Parts:
- added C10: 0.1uF, Capacitor_THT:C_Disc_D4.3mm_W1.9mm_P5.00mm, F.Cu at (154.9, 92.1)
- C1: value C -> 0.8uF
- C2: value C -> 0.4uF
- C4: value C -> 0.2uF
- C5, C6: value C -> 0.1uF
Connections:
- J1 pad 4: /OUT -> Net-(C10-Pad2)
Routing:
- net /OUT: track 54.5 -> 44.1 mm
- net Net-(C10-Pad2): track 0.00 -> 5.32 mm
